Commit message: Reflected the changes to the KrangBlocks

File: etc/model/KrangBlocks.urdf (robot description, URDF)
Before this commit: robot Krang, 26 links, 25 joints
Links:
- link Spine: geometry collision box size=0.134 0.60 0.133; collision box size=0.435 0.16 0.135
Joints:
- joint JKinect: origin xyz=-0.001 0.1805 -0.1120 rpy=3.1416 0 0 -> xyz=-0.000 0.0985 -0.1120 rpy=2.5416 0 0; type revolute -> fixed
- joint JTorso: origin xyz=-0.0285 0.584 0.1088 rpy=0 3.1416 0 -> xyz=-0.0270 0.6670 0.1088 rpy=0 3.1416 0
- joint LJ1: origin xyz=0.2823 0.0845 0 rpy=0 3.1416 -1.5708 -> xyz=0.2823 0.000 0 rpy=0 3.1416 -1.5708
- joint RJ1: origin xyz=-0.2823 0.0845 0 rpy=0 0 1.5708 -> xyz=-0.2823 0.0 0 rpy=0 0 1.5708
