Commit message: Separated the collision for the spine into two boxes

File: etc/model/Krang.urdf (robot description, URDF)
Before this commit: robot Krang, 24 links, 23 joints
Links:
- link Base: geometry collision box size=0.620 0.66 0.329; visual mesh filename=base.dae
- link Spine: geometry collision box size=0.134 0.60 0.133; collision box size=0.435 0.16 0.135

File: etc/model/KrangBlocks.urdf (robot description, URDF)
Before this commit: robot Krang, 24 links, 23 joints
Links:
- link Spine: geometry collision box size=0.134 0.60 0.133; collision box size=0.235 0.16 0.135

Commit message: Created the cylinder collision shape for the wheels

File: etc/model/Krang.urdf (robot description, URDF)
Before this commit: robot Krang, 24 links, 23 joints
Links:
- link LWheel: geometry collision cylinder length=0.077 radius=0.268; visual mesh filename=../model/wheel.dae
- link RWheel: geometry collision cylinder length=0.077 radius=0.268; visual mesh filename=../model/wheel.dae

Commit message: We have hands!

File: etc/model/Krang.urdf (robot description, URDF)
Before this commit: robot Krang, 24 links, 23 joints
Links:
- removed link lgPlate1
- removed link lgPlate2
- removed link rgPlate1
- removed link rgPlate2
- added link lFingerA, mass 0.0001; visual mesh filename=Schunk/finger.dae
- added link lFingerB, mass 0.0001; visual mesh filename=Schunk/finger.dae
- added link lFingerC, mass 0.0001; visual mesh filename=Schunk/finger.dae
- added link rFingerA, mass 0.0001; visual mesh filename=Schunk/finger.dae
- added link rFingerB, mass 0.0001; visual mesh filename=Schunk/finger.dae
- added link rFingerC, mass 0.0001; visual mesh filename=Schunk/finger.dae
Joints:
- removed joint LMotorPlate1
- removed joint LMotorPlate2
- removed joint RMotorPlate1
- removed joint RMotorPlate2
- added joint LJFA: type revolute, parent lGripper, child lFingerA, origin xyz=0.004 0.040 0.127 rpy=3.1416 0.8 1.5708, axis 0 -1 0, limit lower=0.0 upper=1.9 effort=1000 velocity=0.1
- added joint LJFB: type revolute, parent lGripper, child lFingerB, origin xyz=0.030 -0.040 0.127 rpy=0 2.4 1.5708, axis 0 -1 0, limit lower=0.0 upper=1.9 effort=1000 velocity=0.1
- added joint LJFC: type revolute, parent lGripper, child lFingerC, origin xyz=-0.035 -0.040 0.127 rpy=0 2.4 1.5708, axis 0 -1 0, limit lower=0.0 upper=1.9 effort=1000 velocity=0.1
- added joint RJFA: type revolute, parent rGripper, child rFingerA, origin xyz=0.004 0.040 0.127 rpy=3.1416 0.8 1.5708, axis 0 -1 0, limit lower=0.0 upper=1.9 effort=1000 velocity=0.1
- added joint RJFB: type revolute, parent rGripper, child rFingerB, origin xyz=0.030 -0.040 0.127 rpy=0 2.40 1.5708, axis 0 -1 0, limit lower=0.0 upper=1.9 effort=1000 velocity=0.1
- added joint RJFC: type revolute, parent rGripper, child rFingerC, origin xyz=-0.035 -0.040 0.127 rpy=0 2.40 1.5708, axis 0 -1 0, limit lower=0.0 upper=1.9 effort=1000 velocity=0.1

File: etc/model/KrangBlocks.urdf (robot description, URDF)
Before this commit: robot Krang, 24 links, 23 joints
Links:
- link Base: geometry collision box size=0.620 0.66 0.329; visual box size=0.620 0.66 0.329
- link LWheel: geometry collision cylinder length=0.077 radius=0.268; visual cylinder length=0.077 radius=0.268
- link RWheel: geometry collision cylinder length=0.077 radius=0.268; visual cylinder length=0.077 radius=0.268

Commit message: Fixed the inertia values of the fingers

File: etc/model/Krang.urdf (robot description, URDF)
Before this commit: robot Krang, 26 links, 25 joints
Joints:
- joint LJFA: origin xyz=0.004 0.040 0.127 rpy=3.1416 0.8 1.5708 -> xyz=0.004 0.040 0.127 rpy=3.1416 1.0 1.5708
- joint LJFB: origin xyz=0.030 -0.040 0.127 rpy=0 2.4 1.5708 -> xyz=0.030 -0.040 0.127 rpy=0 2.3 1.5708
- joint LJFC: origin xyz=-0.035 -0.040 0.127 rpy=0 2.4 1.5708 -> xyz=-0.035 -0.040 0.127 rpy=0 2.3 1.5708
- joint RJFA: origin xyz=0.004 0.040 0.127 rpy=3.1416 0.8 1.5708 -> xyz=0.004 0.040 0.127 rpy=3.1416 1.0 1.5708
- joint RJFB: origin xyz=0.030 -0.040 0.127 rpy=0 2.40 1.5708 -> xyz=0.030 -0.040 0.127 rpy=0 2.30 1.5708
- joint RJFC: origin xyz=-0.035 -0.040 0.127 rpy=0 2.40 1.5708 -> xyz=-0.035 -0.040 0.127 rpy=0 2.30 1.5708

Commit message: Adding the collision model for the finger

File: etc/model/Krang.urdf (robot description, URDF)
Before this commit: robot Krang, 26 links, 25 joints
Links:
- link lFingerA: geometry collision mesh filename=Schunk/finger.dae; visual mesh filename=Schunk/finger.dae
- link lFingerB: geometry collision mesh filename=Schunk/finger.dae; visual mesh filename=Schunk/finger.dae
- link lFingerC: geometry collision mesh filename=Schunk/finger.dae; visual mesh filename=Schunk/finger.dae
- link lGripper: geometry collision box size=0.15 0.125 0.210; visual mesh filename=Schunk/L7.dae
- link rFingerA: geometry collision mesh filename=Schunk/finger.dae; visual mesh filename=Schunk/finger.dae
- link rFingerB: geometry collision mesh filename=Schunk/finger.dae; visual mesh filename=Schunk/finger.dae
- link rFingerC: geometry collision mesh filename=Schunk/finger.dae; visual mesh filename=Schunk/finger.dae
- link rGripper: geometry collision box size=0.15 0.125 0.210; visual mesh filename=Schunk/L7.dae

Commit message: Got the collision boxes for the fingers

File: etc/model/Krang.urdf (robot description, URDF)
Before this commit: robot Krang, 26 links, 25 joints
Links:
- link lFingerA: geometry collision box size=0.035 0.049 0.0356; collision box size=0.035 0.07 0.0366
- link lFingerB: geometry collision box size=0.035 0.049 0.0356; collision box size=0.035 0.07 0.0366
- link lFingerC: geometry collision box size=0.035 0.049 0.0356; collision box size=0.035 0.07 0.0366
- link rFingerA: geometry collision box size=0.035 0.049 0.0356; collision box size=0.035 0.07 0.0366
- link rFingerB: geometry collision box size=0.035 0.049 0.0356; collision box size=0.035 0.07 0.0366
- link rFingerC: geometry collision box size=0.035 0.049 0.0356; collision box size=0.035 0.07 0.0366

Commit message: Updated the changes to KrangBlocks

File: etc/model/Krang.urdf (robot description, URDF)
Before this commit: robot Krang, 26 links, 25 joints
Joints:
- joint LJ1: limit lower=-3.1416 upper=3.1416 effort=1000 velocity=0.1 -> lower=-4.7124 upper=4.7124 effort=1000 velocity=0.1
- joint LJFT: origin xyz=0 -0.200 0 rpy=1.5708 4.7124 0 -> xyz=0 -0.200 0 rpy=1.5708 3.1416 0
- joint RJFT: origin xyz=0 -0.200 0 rpy=1.5708 4.7124 0 -> xyz=0 -0.200 0 rpy=1.5708 3.1416 0

File: etc/model/KrangBlocks.urdf (robot description, URDF)
Before this commit: robot Krang, 24 links, 23 joints
Links:
- removed link lgPlate1
- removed link lgPlate2
- removed link rgPlate1
- removed link rgPlate2
- added link lFingerA, mass 0.0001; collision box size=0.035 0.049 0.0356; collision box size=0.035 0.07 0.0366
- added link lFingerB, mass 0.0001; collision box size=0.035 0.049 0.0356; collision box size=0.035 0.07 0.0366
- added link lFingerC, mass 0.0001; collision box size=0.035 0.049 0.0356; collision box size=0.035 0.07 0.0366
- added link rFingerA, mass 0.0001; collision box size=0.035 0.049 0.0356; collision box size=0.035 0.07 0.0366
- added link rFingerB, mass 0.0001; collision box size=0.035 0.049 0.0356; collision box size=0.035 0.07 0.0366
- added link rFingerC, mass 0.0001; collision box size=0.035 0.049 0.0356; collision box size=0.035 0.07 0.0366
- link lGripper: geometry collision box size=0.15 0.125 0.210; visual box size=0.15 0.125 0.210
- link rGripper: geometry collision box size=0.15 0.125 0.210; visual box size=0.15 0.125 0.210
Joints:
- removed joint LMotorPlate1
- removed joint LMotorPlate2
- removed joint RMotorPlate1
- removed joint RMotorPlate2
- added joint LJFA: type revolute, parent lGripper, child lFingerA, origin xyz=0.004 0.040 0.127 rpy=3.1416 1.0 1.5708, axis 0 -1 0, limit lower=0.0 upper=1.9 effort=1000 velocity=0.1
- added joint LJFB: type revolute, parent lGripper, child lFingerB, origin xyz=0.030 -0.040 0.127 rpy=0 2.3 1.5708, axis 0 -1 0, limit lower=0.0 upper=1.9 effort=1000 velocity=0.1
- added joint LJFC: type revolute, parent lGripper, child lFingerC, origin xyz=-0.035 -0.040 0.127 rpy=0 2.3 1.5708, axis 0 -1 0, limit lower=0.0 upper=1.9 effort=1000 velocity=0.1
- added joint RJFA: type revolute, parent rGripper, child rFingerA, origin xyz=0.004 0.040 0.127 rpy=3.1416 1.0 1.5708, axis 0 -1 0, limit lower=0.0 upper=1.9 effort=1000 velocity=0.1
- added joint RJFB: type revolute, parent rGripper, child rFingerB, origin xyz=0.030 -0.040 0.127 rpy=0 2.30 1.5708, axis 0 -1 0, limit lower=0.0 upper=1.9 effort=1000 velocity=0.1
- added joint RJFC: type revolute, parent rGripper, child rFingerC, origin xyz=-0.035 -0.040 0.127 rpy=0 2.30 1.5708, axis 0 -1 0, limit lower=0.0 upper=1.9 effort=1000 velocity=0.1
- joint LJ1: limit lower=-3.1416 upper=3.1416 effort=1000 velocity=0.1 -> lower=-4.7124 upper=4.7124 effort=1000 velocity=0.1
- joint LJ3: limit lower=-3.1416 upper=3.1416 effort=1000 velocity=0.1 -> lower=-4.7124 upper=4.7124 effort=1000 velocity=0.1
- joint LJ5: limit lower=-3.1416 upper=3.1416 effort=1000 velocity=0.1 -> lower=-4.7124 upper=4.7124 effort=1000 velocity=0.1
- joint LJFT: limit lower=-3.1416 upper=3.1416 effort=1000 velocity=0.1 -> lower=-4.7124 upper=4.7124 effort=1000 velocity=0.1
- joint RJ1: limit lower=-3.1416 upper=3.1416 effort=1000 velocity=0.1 -> lower=-4.7124 upper=4.7124 effort=1000 velocity=0.1
- joint RJ3: limit lower=-3.1416 upper=3.1416 effort=1000 velocity=0.1 -> lower=-4.7124 upper=4.7124 effort=1000 velocity=0.1
- joint RJ5: limit lower=-3.1416 upper=3.1416 effort=1000 velocity=0.1 -> lower=-4.7124 upper=4.7124 effort=1000 velocity=0.1
- joint RJFT: limit lower=-3.1416 upper=3.1416 effort=1000 velocity=0.1 -> lower=-4.7124 upper=4.7124 effort=1000 velocity=0.1

Commit message: Created the scene to grasp an object from a table

File: etc/model/Krang.urdf (robot description, URDF)
Before this commit: robot Krang, 26 links, 25 joints
Joints:
- joint JKinect: origin xyz=-0.001 0.1805 -0.1120 rpy=3.1416 0 0 -> xyz=-0.001 0.1805 -0.1120 rpy=2.5416 0 0; type revolute -> fixed

Commit message: Changed the center of the bracket and moved the joints for it

File: etc/model/Krang.urdf (robot description, URDF)
Before this commit: robot Krang, 26 links, 25 joints
Joints:
- joint JKinect: origin xyz=-0.001 0.1805 -0.1120 rpy=2.5416 0 0 -> xyz=-0.000 0.0985 -0.1120 rpy=2.5416 0 0
- joint JTorso: origin xyz=-0.0285 0.584 0.1088 rpy=0 3.1416 0 -> xyz=-0.0270 0.6670 0.1088 rpy=0 3.1416 0
- joint LJ1: origin xyz=0.2823 0.0845 0 rpy=0 3.1416 -1.5708 -> xyz=0.2823 0.000 0 rpy=0 3.1416 -1.5708
- joint RJ1: origin xyz=-0.2823 0.0845 0 rpy=0 0 1.5708 -> xyz=-0.2823 0.0 0 rpy=0 0 1.5708

Commit message: Increased the precision of pi

File: etc/model/Krang.urdf (robot description, URDF)
Before this commit: robot Krang, 26 links, 25 joints
Joints:
- joint LJ1: origin xyz=0.2823 0.000 0 rpy=0 3.1416 -1.5708 -> xyz=0.2823 0.000 0 rpy=0 3.141592 -1.570796
- joint LJ2: origin xyz=0 0.0 0 rpy=3.14 3.14 0 -> xyz=0 0.0 0 rpy=3.141592 3.141592 0
- joint LJ3: origin xyz=0 -0.328 0 rpy=-3.1416 -3.1416 0 -> xyz=0 -0.328 0 rpy=-3.141592 -3.141592 0
- joint LJ4: origin xyz=0 0 0 rpy=3.1416 3.1416 0 -> xyz=0 0 0 rpy=3.141592 3.141592 0
- joint LJ5: origin xyz=0 -0.2765 0 rpy=3.1416 3.1416 0 -> xyz=0 -0.2765 0 rpy=3.141592 3.141592 0
- joint LJ6: origin xyz=0 0.0 0 rpy=3.1416 3.1416 0 -> xyz=0 0.0 0 rpy=3.141592 3.141592 0
- joint LJFT: origin xyz=0 -0.200 0 rpy=1.5708 3.1416 0 -> xyz=0 -0.200 0 rpy=1.570796 3.141592 0
- joint RJ1: origin xyz=-0.2823 0.0 0 rpy=0 0 1.5708 -> xyz=-0.2823 0.0 0 rpy=0 0 1.570796
- joint RJ2: origin xyz=0 0.0 0 rpy=3.14 3.14 0 -> xyz=0 0.0 0 rpy=3.141592 3.141592 0
- joint RJ3: origin xyz=0 -0.328 0 rpy=-3.1416 -3.1416 0 -> xyz=0 -0.328 0 rpy=-3.141592 -3.141592 0
- joint RJ4: origin xyz=0 0 0 rpy=3.1416 3.1416 0 -> xyz=0 0 0 rpy=3.141592 3.141592 0
- joint RJ5: origin xyz=0 -0.2765 0 rpy=3.1416 3.1416 0 -> xyz=0 -0.2765 0 rpy=3.141592 3.141592 0
- joint RJ6: origin xyz=0 0.0 0 rpy=3.1416 3.1416 0 -> xyz=0 0.0 0 rpy=3.141592 3.141592 0
- joint RJFT: origin xyz=0 -0.200 0 rpy=1.5708 3.1416 0 -> xyz=0 -0.200 0 rpy=1.570796 3.141592 0

Commit message: Made the Kinect dof revolute as opposed to fixed to make sure f/t estimation works

File: etc/model/Krang.urdf (robot description, URDF)
Before this commit: robot Krang, 26 links, 25 joints
Joints:
- joint JKinect: type fixed -> revolute

File: etc/model/KrangBlocks.urdf (robot description, URDF)
Before this commit: robot Krang, 26 links, 25 joints
Joints:
- joint JKinect: type fixed -> revolute

Commit message: Reflected the changes to the mass and com values to the urdf values (see com report) and wrapped the lines on urdf files to 100 chars

File: etc/model/Krang.urdf (robot description, URDF)
Before this commit: robot Krang, 26 links, 25 joints
Links:
- link Base: mass 81.856 -> 75.767
- link Bracket: mass 10.17 -> 0.17
- link L1: mass 3.836 -> 3.952
- link L2: mass 2.385 -> 3.925
- link L3: mass 2.306 -> 2.373
- link L4: mass 1.477 -> 2.373
- link L5: mass 1.369 -> 1.41334
- link L6: mass 1.47 -> 2.64634
- link R1: mass 3.836 -> 3.952
- link R2: mass 2.385 -> 3.925
- link R3: mass 2.306 -> 2.373
- link R4: mass 1.477 -> 2.373
- link R5: mass 1.369 -> 1.41334
- link R6: mass 1.47 -> 2.64634
- link Spine: mass 10.302 -> 14.006

File: etc/model/KrangBlocks.urdf (robot description, URDF)
Before this commit: robot Krang, 26 links, 25 joints
Links:
- link Base: mass 81.856 -> 75.767
- link Bracket: mass 10.17 -> 0.17
- link L1: mass 3.836 -> 3.952
- link L2: mass 2.385 -> 3.925
- link L3: mass 2.306 -> 2.373
- link L4: mass 1.477 -> 2.373
- link L5: mass 1.369 -> 1.41334
- link L6: mass 1.47 -> 2.64634
- link R1: mass 3.836 -> 3.952
- link R2: mass 2.385 -> 3.925
- link R3: mass 2.306 -> 2.373
- link R4: mass 1.477 -> 2.373
- link R5: mass 1.369 -> 1.41334
- link R6: mass 1.47 -> 2.64634
- link Spine: mass 10.302 -> 14.006
Joints:
- joint LJ1: origin xyz=0.2823 0.000 0 rpy=0 3.1416 -1.5708 -> xyz=0.2823 0.000 0 rpy=0 3.141592 -1.570796
- joint LJ2: origin xyz=0 0.0 0 rpy=3.14 3.14 0 -> xyz=0 0.0 0 rpy=3.141592 3.141592 0
- joint LJ3: origin xyz=0 -0.328 0 rpy=-3.1416 -3.1416 0 -> xyz=0 -0.328 0 rpy=-3.141592 -3.141592 0
- joint LJ4: origin xyz=0 0 0 rpy=3.1416 3.1416 0 -> xyz=0 0 0 rpy=3.141592 3.141592 0
- joint LJ5: origin xyz=0 -0.2765 0 rpy=3.1416 3.1416 0 -> xyz=0 -0.2765 0 rpy=3.141592 3.141592 0
- joint LJ6: origin xyz=0 0 0 rpy=3.1416 3.1416 0 -> xyz=0 0.0 0 rpy=3.141592 3.141592 0
- joint LJFT: origin xyz=0 -0.200 0 rpy=1.5708 3.1416 0 -> xyz=0 -0.200 0 rpy=1.570796 3.141592 0
- joint RJ1: origin xyz=-0.2823 0.0 0 rpy=0 0 1.5708 -> xyz=-0.2823 0.0 0 rpy=0 0 1.570796
- joint RJ2: origin xyz=0 0.0 0 rpy=3.14 3.14 0 -> xyz=0 0.0 0 rpy=3.141592 3.141592 0
- joint RJ3: origin xyz=0 -0.328 0 rpy=-3.1416 -3.1416 0 -> xyz=0 -0.328 0 rpy=-3.141592 -3.141592 0
- joint RJ4: origin xyz=0 0 0 rpy=3.1416 3.1416 0 -> xyz=0 0 0 rpy=3.141592 3.141592 0
- joint RJ5: origin xyz=0 -0.2765 0 rpy=3.1416 3.1416 0 -> xyz=0 -0.2765 0 rpy=3.141592 3.141592 0
- joint RJ6: origin xyz=0 0 0 rpy=3.1416 3.1416 0 -> xyz=0 0.0 0 rpy=3.141592 3.141592 0
- joint RJFT: origin xyz=0 -0.200 0 rpy=1.5708 3.1416 0 -> xyz=0 -0.200 0 rpy=1.570796 3.141592 0

Commit message: Added the new tilt/pan kinect.

File: etc/model/Krang.urdf (robot description, URDF)
Before this commit: robot Krang, 26 links, 25 joints
Links:
- added link TiltMotor, mass 0.705; collision box size=0.28 0.07 0.063; visual mesh filename=tilt.dae
Joints:
- removed joint JKinect
- added joint JPan: type revolute, parent Bracket, child TiltMotor, origin xyz=-0.0015 0.0755 -0.071 rpy=2.5416 0 -1.5708, axis 1 0 0, limit lower=-3.1416 upper=3.1416 effort=1000 velocity=0.1
- added joint JTilt: type revolute, parent TiltMotor, child Kinect, origin xyz=-0.042 0.0 0.0055 rpy=0 0 1.5708, axis 1 0 0, limit lower=-3.1416 upper=3.1416 effort=1000 velocity=0.1

File: etc/model/KrangBlocks.urdf (robot description, URDF)
Before this commit: robot Krang, 26 links, 25 joints
Links:
- added link TiltMotor, mass 0.705; collision box size=0.28 0.07 0.063; visual mesh filename=tilt.dae
- link Kinect: geometry collision box size=0.28 0.07 0.063; visual mesh filename=kinect.dae
Joints:
- removed joint JKinect
- added joint JPan: type revolute, parent Bracket, child TiltMotor, origin xyz=-0.0015 0.0755 -0.071 rpy=2.5416 0 -1.5708, axis 1 0 0, limit lower=-3.1416 upper=3.1416 effort=1000 velocity=0.1
- added joint JTilt: type revolute, parent TiltMotor, child Kinect, origin xyz=-0.042 0.0 0.0055 rpy=0 0 1.5708, axis 1 0 0, limit lower=-3.1416 upper=3.1416 effort=1000 velocity=0.1

Commit message: Set the default value for the pan axis

File: etc/model/Krang.urdf (robot description, URDF)
Before this commit: robot Krang, 27 links, 26 joints
Joints:
- joint JPan: origin xyz=-0.0015 0.0755 -0.071 rpy=2.5416 0 -1.5708 -> xyz=-0.0015 0.0755 -0.071 rpy=0 0 -1.5708

File: etc/model/KrangBlocks.urdf (robot description, URDF)
Before this commit: robot Krang, 27 links, 26 joints
Joints:
- joint JPan: origin xyz=-0.0015 0.0755 -0.071 rpy=2.5416 0 -1.5708 -> xyz=-0.0015 0.0755 -0.071 rpy=0 0 -1.5708

Commit message: Rotated the tilt motor 90 degrees

File: etc/model/Krang.urdf (robot description, URDF)
Before this commit: robot Krang, 27 links, 26 joints
Joints:
- joint JPan: origin xyz=-0.0015 0.0755 -0.071 rpy=0 0 -1.5708 -> xyz=-0.0015 0.0755 -0.071 rpy=3.1416 0 -1.5708
- joint JTilt: origin xyz=-0.042 0.0 0.0055 rpy=0 0 1.5708 -> xyz=-0.0702 0.0 -0.0067 rpy=0 3.1416 1.5708

File: etc/model/KrangBlocks.urdf (robot description, URDF)
Before this commit: robot Krang, 27 links, 26 joints
Joints:
- joint JPan: origin xyz=-0.0015 0.0755 -0.071 rpy=0 0 -1.5708 -> xyz=-0.0015 0.0755 -0.071 rpy=3.1416 0 -1.5708
- joint JTilt: origin xyz=-0.042 0.0 0.0055 rpy=0 0 1.5708 -> xyz=-0.0702 0.0 -0.0067 rpy=0 3.1416 1.5708

Commit message: Moved Krang to the floor and changed axis of rotation of tilt axis

File: etc/model/Krang.urdf (robot description, URDF)
Before this commit: robot Krang, 27 links, 26 joints
Joints:
- joint JTilt: axis 1 0 0 -> -1 0 0

File: etc/model/KrangBlocks.urdf (robot description, URDF)
Before this commit: robot Krang, 27 links, 26 joints
Joints:
- joint JTilt: axis 1 0 0 -> -1 0 0

Commit message: Moved all the robot configurations to 0.267 height to stop collisions with ground and set the collision box for new kinect

File: etc/model/Krang.urdf (robot description, URDF)
Before this commit: robot Krang, 27 links, 26 joints
Links:
- link Kinect: geometry collision box size=0.3 0.1 0.1; visual mesh filename=kinect.dae
- link TiltMotor: geometry collision box size=0.01 0.01 0.01; visual mesh filename=tilt.dae

Commit message: Enlarged the collision boxes

File: etc/model/Krang.urdf (robot description, URDF)
Before this commit: robot Krang, 27 links, 26 joints
Links:
- link L1: geometry collision box size=0.16 0.33 0.18; visual mesh filename=Schunk/L1.dae
- link L2: geometry collision box size=0.19 0.29 0.18; visual mesh filename=Schunk/L2.dae
- link L3: geometry collision box size=0.1800 0.31 0.16; visual mesh filename=Schunk/L3.dae
- link L4: geometry collision box size=0.17 0.25 0.16; visual mesh filename=Schunk/L4.dae
- link L5: geometry collision box size=0.18 0.26 0.13; visual mesh filename=Schunk/L5.dae
- link L6: geometry collision box size=0.17 0.21 0.13; visual mesh filename=Schunk/L6.dae
- link lFingerA: geometry collision box size=0.07 0.10 0.07; collision box size=0.07 0.10 0.07
- link lFingerB: geometry collision box size=0.07 0.10 0.07; collision box size=0.07 0.10 0.07
- link lFingerC: geometry collision box size=0.07 0.10 0.07; collision box size=0.07 0.10 0.07
- link lGripper: geometry collision box size=0.21 0.19 0.270; visual mesh filename=Schunk/L7.dae

Commit message: Removed larger collision boxes

File: etc/model/Krang.urdf (robot description, URDF)
Before this commit: robot Krang, 27 links, 26 joints
Links:
- link L3: geometry collision box size=0.13800 0.26217 0.11189; visual mesh filename=Schunk/L3.dae
- link L4: geometry collision box size=0.12960 0.2141 0.11; visual mesh filename=Schunk/L4.dae
- link L5: geometry collision box size=0.117977 0.204179 0.089915; visual mesh filename=Schunk/L5.dae
- link L6: geometry collision box size=0.111977 0.185277 0.089; visual mesh filename=Schunk/L6.dae
- link lGripper: geometry collision box size=0.15 0.125 0.210; visual mesh filename=Schunk/L7.dae

Commit message: Removed the bigger collision boxes from l1 and l2 as well

File: etc/model/Krang.urdf (robot description, URDF)
Before this commit: robot Krang, 27 links, 26 joints
Links:
- link L1: geometry collision box size=0.16 0.29367 0.13188; visual mesh filename=Schunk/L1.dae
- link L2: geometry collision box size=0.14591 0.24658 0.13; visual mesh filename=Schunk/L2.dae
